Commit message: fixed tf issues and now can visualise robot model in rviz2

File: urdfs/vnymous.urdf (robot description, URDF)
Before this commit: robot vikram, 9 links, 8 joints
Links:
- link base_link: geometry collision mesh filename=file:///home/tamoghna/ros2_ws/src/vsim/meshes/igvc/igvc_bot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 scale=0.001 0.001 0.001; visual mesh filename=file:///home/tamoghna/ros2_ws/src/vsim/meshes/igvc/igvc_bot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 scale=0.001 0.001 0.001
- link wheel1: geometry collision cylinder length=0.04 radius=0.12; visual mesh filename=file:///home/tamoghna/ros2_ws/src/vsim/meshes/igvc/igvc_whe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 scale=0.001 0.001 0.001
- link wheel2: geometry collision cylinder length=0.04 radius=0.12; visual mesh filename=file:///home/tamoghna/ros2_ws/src/vsim/meshes/igvc/igvc_whe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 scale=0.001 0.001 0.001
- link zed_camera: geometry collision mesh filename=file:///home/tamoghna/ros2_ws/src/vsim/meshes/igvc/zed2i.dae; visual mesh filename=file:///home/tamoghna/ros2_ws/src/vsim/meshes/igvc/zed2i.dae scale=1 1 1
Joints:
- joint camera_to_body: origin xyz=-0.02 0.13 0.905 rpy=0 0 1.57 -> xyz=-0.02 0.13 0.905 rpy=0 0 1.5707
- joint perp: origin xyz=0.15 0 1.58 rpy=-1.5707 0 -1.5707 -> xyz=-0.02 0.13 0.905 rpy=-1.5707 0 -1.5707

Commit message: made minor changes

File: urdfs/vnymous.urdf (robot description, URDF)
Before this commit: robot vnymous, 9 links, 8 joints
Joints:
- joint perp: origin xyz=-0.02 0.13 0.905 rpy=-1.5707 0 -1.5707 -> xyz=-0.02 0.13 0.905 rpy=-1.5707 0 0

Commit message: corrected cmd_vel and odom tfs

File: urdfs/vnymous.urdf (robot description, URDF)
Before this commit: robot vnymous, 9 links, 8 joints
Joints:
- removed joint camera_to_body
- added joint body_to_cam: type fixed, parent base_link, child zed_camera, origin xyz=0.14 0.02 0.905 rpy=0 0 0
- joint body_to_castor_cylinder: origin xyz=0.002746 -0.377785 -0.01 rpy=0 0 0 -> xyz=-0.37 0 0 rpy=0 0 0
- joint body_to_castor_cylinder2: origin xyz=0.002746 0.377785 0 rpy=0 0 0 -> xyz=0.37 0 -0.01 rpy=0 0 0
- joint body_to_wheel1: origin xyz=0.2 0.0 0 rpy=0 0 3.14 -> xyz=0.0 -0.21 0 rpy=0 0 1.5707
- joint body_to_wheel2: origin xyz=-0.22 0.0 0 rpy=0 0 0 -> xyz=-0.005 0.22 0 rpy=0 0 -1.5707
- joint perp: origin xyz=-0.02 0.13 0.905 rpy=-1.5707 0 0 -> xyz=-0.02 0.13 0.905 rpy=-1.5707 0 -1.5707

Commit message: nothing works

File: urdfs/vnymous.urdf (robot description, URDF)
Before this commit: robot vnymous, 9 links, 8 joints
Links:
- added link gps_link, mass 0.5; collision box size=0.1 0.1 0.1; visual box size=0.1 0.1 0.1
- link perpendicular: mass 0 -> 0.1; geometry collision box size=0.001 0.001 0.001; visual box size=0.001 0.001 0.001
Joints:
- removed joint perp
- added joint body_to_gps: type fixed, parent base_link, child gps_link, origin xyz=0 0 0.25 rpy=0 0 0
- added joint body_to_perpendicular: type fixed, parent base_link, child perpendicular, origin xyz=0.14 0.02 0.905 rpy=-1.5707 0 -1.5707

Commit message: everything works

File: urdfs/vnymous.urdf (robot description, URDF)
Before this commit: robot vnymous, 10 links, 9 joints
Links:
- link gps_link: geometry collision box size=0.13 0.13 0.07; visual box size=0.13 0.13 0.07
- link perpendicular: mass 0.1 -> 0; geometry collision box size=0.0001 0.00001 0.00001; visual box size=0.0001 0.00001 0.00001
Joints:
- removed joint body_to_perpendicular
- added joint perp: type fixed, parent base_link, child perpendicular, origin xyz=-0.02 0.13 0.905 rpy=-1.5707 0 -1.5707
- joint body_to_gps: origin xyz=0 0 0.25 rpy=0 0 0 -> xyz=-0.26 0 0.275 rpy=0 0 0

Commit message: modified for gps

File: urdfs/vnymous.urdf (robot description, URDF)
Before this commit: robot vnymous, 10 links, 9 joints
Links:
- added link base_footprint
- added link imu_link, mass 0.2; collision box size=0.1 0.1 0.07; visual box size=0.1 0.1 0.07
Joints:
- added joint body_to_imu: type fixed, parent base_link, child imu_link, origin xyz=-0.1 0 0.275 rpy=0 0 0
- added joint footprint_to_baselink: type fixed, parent base_footprint, child base_link, origin xyz=0 0 0 rpy=0 0 0.010
